File: ESP12E.3.sch (KiCad schematic (older format))
At the start: 30 parts, among them Q1 MOSFET-NREFLOW, U1 SPX3819M5-L-3-3, X1 ESP-12

Commit message: Update to net assignments and part updates.
Parts:
- JP1, JP10, JP11, JP2, JP3, JP4, JP9: symbol ESP12E.3-eagle-import:PINHD-1X3 -> Connector:Conn_01x03_Male
Connections:
- net labels added: GPIO16
- net labels removed: VCC
- wire segments 70 -> 82
Changed lines of the file:
@@
 Text Label 4700 2300 0    70   ~ 0
 GND
-Wire Wire Line
-	8200 1800 8200 2700
-Text Label 8200 1800 0    10   ~ 0
-GND
-Wire Wire Line
-	6700 3000 6800 3000
-Wire Wire Line
-	6800 3000 7000 3000
-Connection ~ 6800 3000
-Text Label 6700 3000 0    10   ~ 0
+Text Label 8000 1800 0    10   ~ 0
 GND
 Wire Wire Line
@@
 Text Label 4700 1900 0    70   ~ 0
 GPIO5
-Wire Wire Line
-	10100 7600 10100 9000
-Text Label 10100 7600 1    70   ~ 0
+Text Label 10100 8850 1    70   ~ 0
 GPIO5
-Text Label 2800 2200 0    70   ~ 0
+Text Label 3050 2200 2    70   ~ 0
 GPIO13
-Wire Wire Line
-	8100 7600 8100 9000
-Text Label 8100 7600 1    70   ~ 0
+Text Label 8100 8850 1    70   ~ 0
 GPIO13
 Wire Wire Line
@@
 VMOT
 Wire Wire Line
-	6600 1100 6600 1400
-Text Label 6600 1100 0    10   ~ 0
+	6800 1100 6800 1400
+Text Label 6800 1100 0    10   ~ 0
 +3V3
 Wire Wire Line
@@
 Text Label 7700 1100 0    10   ~ 0
 +3V3
-Text Label 2800 2300 0    70   ~ 0
+Text Label 3050 2300 2    70   ~ 0
 +3V3
 Wire Wire Line
@@
 +3V3
 Wire Wire Line
-	8200 1400 8200 1100
-Text Label 8200 1100 0    70   ~ 0
+	8000 1400 8000 1100
+Text Label 8000 1100 0    70   ~ 0
 GPIO15
 Text Label 4700 2200 0    70   ~ 0
 GPIO15
-Text Label 2800 2100 0    70   ~ 0
+Text Label 3050 2100 2    70   ~ 0
 GPIO12
-Wire Wire Line
-	8700 7600 8700 9000
-Text Label 8700 7600 1    70   ~ 0
+Text Label 8700 8850 1    70   ~ 0
 GPIO12
-Text Label 2800 2000 0    70   ~ 0
+Text Label 3050 2000 2    70   ~ 0
 GPIO14
-Wire Wire Line
-	9400 9000 9400 7600
-Text Label 9400 7600 1    70   ~ 0
+Text Label 9400 8850 1    70   ~ 0
 GPIO14
-Text Label 2800 1800 0    70   ~ 0
+Text Label 3050 1800 2    70   ~ 0
 CH_PD
 Wire Wire Line
@@
 Text Label 7700 2200 1    70   ~ 0
 CH_PD
-Text Label 2800 1700 0    70   ~ 0
+Text Label 3050 1700 2    70   ~ 0
 ADC
-Text Label 2800 1600 0    70   ~ 0
+Text Label 3050 1600 2    70   ~ 0
 RESET
-Wire Wire Line
-	7000 2400 7100 2400
-Wire Wire Line
-	7100 2400 7100 1800
-Text Label 7100 2100 1    70   ~ 0
+Text Label 7100 2200 1    70   ~ 0
 RESET
 Text Label 4600 6100 0    70   ~ 0
@@
 Text Label 4700 2000 0    70   ~ 0
 GPIO0
-Wire Wire Line
-	6600 2400 6700 2400
-Wire Wire Line
-	6600 1800 6600 2400
-Text Label 6600 2100 1    70   ~ 0
+Text Label 6800 2200 1    70   ~ 0
 GPIO0
 Wire Wire Line
@@
 L ESP12E.3-eagle-import:R-US_R0603 R8
 U 1 0 3097C624
-P 8200 1600
-F 0 "R8" H 8050 1659 59  0000 L BNN
-F 1 "10k" H 8050 1470 59  0000 L BNN
-F 2 "ESP12E.3:R0603" H 8200 1600 50  0001 C CNN
-F 3 "" H 8200 1600 50  0001 C CNN
-	1    8200 1600
+P 8000 1600
+F 0 "R8" H 7850 1659 59  0000 L BNN
+F 1 "10k" H 7850 1470 59  0000 L BNN
+F 2 "ESP12E.3:R0603" H 8000 1600 50  0001 C CNN
+F 3 "" H 8000 1600 50  0001 C CNN
+	1    8000 1600
 	0    -1   -1   0
 $EndComp
@@
 L ESP12E.3-eagle-import:R-US_R0603 R9
 U 1 0 22FF1DF3
-P 6600 1600
-F 0 "R9" H 6450 1659 59  0000 L BNN
-F 1 "10k" H 6450 1470 59  0000 L BNN
-F 2 "ESP12E.3:R0603" H 6600 1600 50  0001 C CNN
-F 3 "" H 6600 1600 50  0001 C CNN
-	1    6600 1600
+P 6800 1600
+F 0 "R9" H 6650 1659 59  0000 L BNN
+F 1 "10k" H 6650 1470 59  0000 L BNN
+F 2 "ESP12E.3:R0603" H 6800 1600 50  0001 C CNN
+F 3 "" H 6800 1600 50  0001 C CNN
+	1    6800 1600
 	0    -1   -1   0
 $EndComp
@@
 L ESP12E.3-eagle-import:+3V3 #+3V01
 U 1 0 7D977A11
-P 6600 1000
-F 0 "#+3V01" H 6600 1000 50  0001 C CNN
-F 1 "+3V3" V 6500 800 59  0000 L BNN
-F 2 "" H 6600 1000 50  0001 C CNN
-F 3 "" H 6600 1000 50  0001 C CNN
-	1    6600 1000
+P 6800 1000
+F 0 "#+3V01" H 6800 1000 50  0001 C CNN
+F 1 "+3V3" V 6700 800 59  0000 L BNN
+F 2 "" H 6800 1000 50  0001 C CNN
+F 3 "" H 6800 1000 50  0001 C CNN
+	1    6800 1000
 	1    0    0    -1
 $EndComp
@@
 $EndComp
 $Comp
-L ESP12E.3-eagle-import:GND #GND07
-U 1 0 C2693486
-P 6800 3100
-F 0 "#GND07" H 6800 3100 50  0001 C CNN
-F 1 "GND" H 6700 3000 59  0000 L BNN
-F 2 "" H 6800 3100 50  0001 C CNN
-F 3 "" H 6800 3100 50  0001 C CNN
-	1    6800 3100
-	1    0    0    -1
-$EndComp
-$Comp
 L ESP12E.3-eagle-import:GND #GND08
 U 1 0 E3161DBF
-P 8200 2800
-F 0 "#GND08" H 8200 2800 50  0001 C CNN
-F 1 "GND" H 8100 2700 59  0000 L BNN
-F 2 "" H 8200 2800 50  0001 C CNN
-F 3 "" H 8200 2800 50  0001 C CNN
-	1    8200 2800
+P 8000 2200
+F 0 "#GND08" H 8000 2200 50  0001 C CNN
+F 1 "GND" H 7900 2100 59  0000 L BNN
+F 2 "" H 8000 2200 50  0001 C CNN
+F 3 "" H 8000 2200 50  0001 C CNN
+	1    8000 2200
 	1    0    0    -1
 $EndComp
@@
 $EndComp
 $Comp
-L ESP12E.3-eagle-import:PINHD-1X3 JP1
+L Connector:Conn_01x03_Male JP1
 U 1 0 0B60073D
-P 10200 9100
-F 0 "JP1" H 9950 9325 59  0000 L BNN
-F 1 "PINHD-1X3" H 9950 8800 59  0000 L BNN
-F 2 "ESP12E.3:1X03" H 10200 9100 50  0001 C CNN
-F 3 "" H 10200 9100 50  0001 C CNN
-	1    10200 9100
-	1    0    0    -1
-$EndComp
-$Comp
-L ESP12E.3-eagle-import:PINHD-1X3 JP2
+P 9900 9100
+F 0 "JP1" H 9650 9325 59  0000 L BNN
+F 1 "PINHD-1X3" H 9650 8800 59  0000 L BNN
+F 2 "ESP12E.3:1X03" H 9900 9100 50  0001 C CNN
+F 3 "" H 9900 9100 50  0001 C CNN
+	1    9900 9100
+	1    0    0    -1
+$EndComp
+$Comp
+L Connector:Conn_01x03_Male JP2
 U 1 0 BAFA783C
-P 9500 9100
-F 0 "JP2" H 9250 9325 59  0000 L BNN
-F 1 "PINHD-1X3" H 9250 8800 59  0000 L BNN
-F 2 "ESP12E.3:1X03" H 9500 9100 50  0001 C CNN
-F 3 "" H 9500 9100 50  0001 C CNN
-	1    9500 9100
-	1    0    0    -1
-$EndComp
-$Comp
-L ESP12E.3-eagle-import:PINHD-1X3 JP3
+P 9200 9100
+F 0 "JP2" H 8950 9325 59  0000 L BNN
+F 1 "PINHD-1X3" H 8950 8800 59  0000 L BNN
+F 2 "ESP12E.3:1X03" H 9200 9100 50  0001 C CNN
+F 3 "" H 9200 9100 50  0001 C CNN
+	1    9200 9100
+	1    0    0    -1
+$EndComp
+$Comp
+L Connector:Conn_01x03_Male JP3
 U 1 0 8182258E
-P 8800 9100
-F 0 "JP3" H 8550 9325 59  0000 L BNN
-F 1 "PINHD-1X3" H 8550 8800 59  0000 L BNN
-F 2 "ESP12E.3:1X03" H 8800 9100 50  0001 C CNN
-F 3 "" H 8800 9100 50  0001 C CNN
-	1    8800 9100
-	1    0    0    -1
-$EndComp
-$Comp
-L ESP12E.3-eagle-import:PINHD-1X3 JP4
+P 8500 9100
+F 0 "JP3" H 8250 9325 59  0000 L BNN
+F 1 "PINHD-1X3" H 8250 8800 59  0000 L BNN
+F 2 "ESP12E.3:1X03" H 8500 9100 50  0001 C CNN
+F 3 "" H 8500 9100 50  0001 C CNN
+	1    8500 9100
+	1    0    0    -1
+$EndComp
+$Comp
+L Connector:Conn_01x03_Male JP4
 U 1 0 193933AB
-P 8200 9100
-F 0 "JP4" H 7950 9325 59  0000 L BNN
-F 1 "PINHD-1X3" H 7950 8800 59  0000 L BNN
-F 2 "ESP12E.3:1X03" H 8200 9100 50  0001 C CNN
-F 3 "" H 8200 9100 50  0001 C CNN
-	1    8200 9100
+P 7900 9100
+F 0 "JP4" H 7650 9325 59  0000 L BNN
+F 1 "PINHD-1X3" H 7650 8800 59  0000 L BNN
+F 2 "ESP12E.3:1X03" H 7900 9100 50  0001 C CNN
+F 3 "" H 7900 9100 50  0001 C CNN
+	1    7900 9100
 	1    0    0    -1
 $EndComp
@@
 $EndComp
 $Comp
-L ESP12E.3-eagle-import:PINHD-1X3 JP10
+L Connector:Conn_01x03_Male JP10
 U 1 0 A1D90C10
-P 11700 4000
-F 0 "JP10" H 11450 4225 59  0000 L BNN
-F 1 "PINHD-1X3" H 11450 3700 59  0000 L BNN
-F 2 "ESP12E.3:1X03" H 11700 4000 50  0001 C CNN
-F 3 "" H 11700 4000 50  0001 C CNN
-	1    11700 4000
-	1    0    0    -1
+P 11800 4000
+F 0 "JP10" H 11550 4225 59  0000 L BNN
+F 1 "PINHD-1X3" H 11550 3700 59  0000 L BNN
+F 2 "ESP12E.3:1X03" H 11800 4000 50  0001 C CNN
+F 3 "" H 11800 4000 50  0001 C CNN
+	1    11800 4000
+	-1   0    0    -1
 $EndComp
 $Comp
@@
 $EndComp
 $Comp
-L ESP12E.3-eagle-import:PINHD-1X3 JP9
+L Connector:Conn_01x03_Male JP9
 U 1 0 C8B46213
+P 4400 6000
+F 0 "JP9" H 4150 6225 59  0000 L BNN
+F 1 "PINHD-1X3" H 4150 5700 59  0000 L BNN
+F 2 "ESP12E.3:1X03" H 4400 6000 50  0001 C CNN
+F 3 "" H 4400 6000 50  0001 C CNN
+	1    4400 6000
+	1    0    0    -1
+$EndComp
+$Comp
+L Connector:Conn_01x03_Male JP11
+U 1 0 E9E46F75
 P 5100 6000
-F 0 "JP9" H 4850 6225 59  0000 L BNN
+F 0 "JP11" H 4850 6225 59  0000 L BNN
 F 1 "PINHD-1X3" H 4850 5700 59  0000 L BNN
 F 2 "ESP12E.3:1X03" H 5100 6000 50  0001 C CNN
 F 3 "" H 5100 6000 50  0001 C CNN
 	1    5100 6000
-	1    0    0    -1
-$EndComp
-$Comp
-L ESP12E.3-eagle-import:PINHD-1X3 JP11
-U 1 0 E9E46F75
-P 5600 6000
-F 0 "JP11" H 5350 6225 59  0000 L BNN
-F 1 "PINHD-1X3" H 5350 5700 59  0000 L BNN
-F 2 "ESP12E.3:1X03" H 5600 6000 50  0001 C CNN
-F 3 "" H 5600 6000 50  0001 C CNN
-	1    5600 6000
 	1    0    0    -1
 $EndComp
@@
 Text Notes 1100 10600 0    59   ~ 0
 " "
-Text GLabel 3200 2300 0    10   BiDi ~ 0
-VCC
 Text GLabel 4600 2300 0    10   BiDi ~ 0
 GND
+Wire Wire Line
+	10100 8850 10100 9000
+Wire Wire Line
+	9400 8850 9400 9000
+Wire Wire Line
+	8700 8850 8700 9000
+Wire Wire Line
+	8100 8850 8100 9000
+Wire Wire Line
+	7100 1800 7100 2200
+Wire Wire Line
+	6800 1800 6800 2200
+Wire Wire Line
+	8000 1800 8000 2100
+Text Label 3050 1900 2    70   ~ 0
+GPIO16
+Wire Wire Line
+	4700 1600 4600 1600
+Wire Wire Line
+	4600 1700 4700 1700
+Wire Wire Line
+	4600 1800 4700 1800
+Wire Wire Line
+	4600 1900 4700 1900
+Wire Wire Line
+	4600 2000 4700 2000
+Wire Wire Line
+	4600 2100 4700 2100
+Wire Wire Line
+	4600 2200 4700 2200
+Wire Wire Line
+	4600 2300 4700 2300
+Wire Wire Line
+	3050 2300 3200 2300
+Wire Wire Line
+	3050 2200 3200 2200
+Wire Wire Line
+	3050 2100 3200 2100
+Wire Wire Line
+	3050 2000 3200 2000
+Wire Wire Line
+	3050 1900 3200 1900
+Wire Wire Line
+	3200 1800 3050 1800
+Wire Wire Line
+	3200 1700 3050 1700
+Wire Wire Line
+	3200 1600 3050 1600
 $EndSCHEMATC
